File: Esp8266_WateringSystem.kicad_pcb (KiCad board)
At the start: 2 copper layers, 105.3 x 97.8 mm, 17 parts, among them J1 Barrel_Jack, J2 PUMP, K2 FINDER-36.11, Q1 NPN, U1 ZC563900, U2 LCD16x2_I2C, U4 L7805, U5 Soil_Moisture_Sensor

Commit message: 28_3_35
Routing:
- net GND: track 4.81 -> 18.6 mm
- net Net-(D1-A): track 71.7 -> 73.1 mm
Changed lines of the file:
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@@
 	)
 	(segment
-		(start 152.8 123.05)
-		(end 152.8 124.3)
-		(width 0.4)
+		(start 152.122182 121.822182)
+		(end 149.6 119.3)
+		(width 0.6)
 		(layer "B.Cu")
 		(net 2)
@@
 	)
 	(segment
+		(start 152.6 125.1)
+		(end 152.3 125.4)
+		(width 0.6)
+		(layer "B.Cu")
+		(net 2)
+	)
+	(segment
 		(start 115.7 139.5)
 		(end 116 139.8)
@@
 	)
 	(segment
+		(start 149.6 111.8)
+		(end 149.6 119.3)
+		(width 0.6)
+		(layer "B.Cu")
+		(net 2)
+	)
+	(segment
 		(start 116 138.6774)
 		(end 116 139.2)
@@
 	)
 	(segment
+		(start 152.9 123.7)
+		(end 152.9 124.375735)
+		(width 0.6)
+		(layer "B.Cu")
+		(net 2)
+	)
+	(segment
 		(start 107.0226 137.8774)
 		(end 107 137.9)
@@
 		(net 2)
 	)
+	(arc
+		(start 152.9 124.375735)
+		(mid 152.822032 124.767704)
+		(end 152.6 125.1)
+		(width 0.6)
+		(layer "B.Cu")
+		(net 2)
+	)
+	(arc
+		(start 152.122182 121.822182)
+		(mid 152.697851 122.683732)
+		(end 152.9 123.7)
+		(width 0.6)
+		(layer "B.Cu")
+		(net 2)
+	)
 	(segment
 		(start 91.95 67.84)
@@
 	)
 	(segment
-		(start 164.4313 100.5446)
-		(end 162.9067 100.5446)
-		(width 0.8)
-		(layer "B.Cu")
-		(net 27)
-	)
-	(segment
 		(start 170.6387 112.6)
 		(end 176.83 112.6)
@@
 	)
 	(segment
-		(start 170.6387 106.752)
-		(end 164.4313 100.5446)
-		(width 0.8)
-		(layer "B.Cu")
-		(net 27)
-	)
-	(segment
-		(start 151.38 113.5)
-		(end 151.38 112.0713)
-		(width 0.8)
-		(layer "B.Cu")
-		(net 27)
-	)
-	(segment
 		(start 170.6387 116.1726)
 		(end 170.6387 112.6)
@@
 	)
 	(segment
-		(start 162.9067 100.5446)
+		(start 165.4 100)
+		(end 163.4513 100)
+		(width 0.8)
+		(layer "B.Cu")
+		(net 27)
+	)
+	(segment
+		(start 163.4513 100)
 		(end 151.38 112.0713)
 		(width 0.8)
@@
 	(segment
 		(start 170.6387 112.6)
-		(end 170.6387 106.752)
+		(end 170.6387 105.2387)
 		(width 0.8)
 		(layer "B.Cu")
@@
 	)
 	(segment
+		(start 151.38 112.0713)
+		(end 151.38 113.5)
+		(width 0.8)
+		(layer "B.Cu")
+		(net 27)
+	)
+	(segment
 		(start 151.38 114.9287)
 		(end 153.9 117.4487)
@@
 	)
 	(segment
+		(start 170.6387 105.2387)
+		(end 165.4 100)
+		(width 0.8)
+		(layer "B.Cu")
+		(net 27)
+	)
+	(segment
 		(start 157.5313 101.7)
 		(end 157.6313 101.8)
@@
 		(hatch edge 0.5)
 		(connect_pads
-			(clearance 0.5)
+			(clearance 0.7)
 		)
 		(min_thickness 0.5)

Commit message: o van ke
Routing:
- net +5V: track 208.1 -> 209.4 mm
Changed lines of the file:
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@@
-	)
-	(segment
-		(start 111.03875 119.73875)
-		(end 97.53875 119.73875)
-		(width 1)
-		(layer "B.Cu")
-		(net 3)
 	)
 	(segment
@@
 	)
 	(segment
+		(start 116 124.7)
+		(end 109.3 118)
+		(width 1)
+		(layer "B.Cu")
+		(net 3)
+	)
+	(segment
 		(start 151 140.1)
 		(end 151 136.1)
@@
 	)
 	(segment
-		(start 97.53875 119.73875)
-		(end 97.4 119.6)
-		(width 1)
-		(layer "B.Cu")
-		(net 3)
-	)
-	(segment
 		(start 169.21 112.6)
 		(end 164.2 112.6)
@@
 	)
 	(segment
+		(start 99 118)
+		(end 97.4 119.6)
+		(width 1)
+		(layer "B.Cu")
+		(net 3)
+	)
+	(segment
 		(start 122.7424 137.1774)
 		(end 116 137.1774)
@@
 	)
 	(segment
+		(start 116 137.1774)
+		(end 116 124.7)
+		(width 1)
+		(layer "B.Cu")
+		(net 3)
+	)
+	(segment
 		(start 97.4 129.2)
 		(end 97.4 119.6)
@@
 	)
 	(segment
-		(start 116 137.1774)
-		(end 116 124.7)
+		(start 109.3 118)
+		(end 99 118)
 		(width 1)
 		(layer "B.Cu")
@@
 	)
 	(segment
-		(start 116 124.7)
-		(end 111.03875 119.73875)
-		(width 1)
-		(layer "B.Cu")
-		(net 3)
-	)
-	(segment
 		(start 91.95 107.45)
 		(end 95.41 110.91)
@@
 	)
 	(segment
-		(start 170.6387 112.6)
-		(end 176.83 112.6)
-		(width 0.8)
-		(layer "B.Cu")
-		(net 27)
-	)
-	(segment
-		(start 164.43 122.3813)
-		(end 170.6387 116.1726)
-		(width 0.8)
-		(layer "B.Cu")
-		(net 27)
-	)
-	(segment
 		(start 153.9 117.4487)
 		(end 153.9 129.2)
@@
 	)
 	(segment
-		(start 170.6387 116.1726)
-		(end 170.6387 112.6)
+		(start 171.7 112.2)
+		(end 171.7 112.6)
 		(width 0.8)
 		(layer "B.Cu")
@@
 	)
 	(segment
+		(start 163.4513 100)
+		(end 165.4 100)
+		(width 0.8)
+		(layer "B.Cu")
+		(net 27)
+	)
+	(segment
 		(start 165.4 100)
-		(end 163.4513 100)
-		(width 0.8)
-		(layer "B.Cu")
-		(net 27)
-	)
-	(segment
-		(start 163.4513 100)
+		(end 171.7 106.3)
+		(width 0.8)
+		(layer "B.Cu")
+		(net 27)
+	)
+	(segment
+		(start 151.38 113.5)
 		(end 151.38 112.0713)
-		(width 0.8)
-		(layer "B.Cu")
-		(net 27)
-	)
-	(segment
-		(start 170.6387 112.6)
-		(end 170.6387 105.2387)
 		(width 0.8)
 		(layer "B.Cu")
@@
 	)
 	(segment
-		(start 164.43 123.66)
+		(start 171.7 115.1113)
 		(end 164.43 122.3813)
 		(width 0.8)
@@
 	)
 	(segment
+		(start 164.43 122.3813)
+		(end 164.43 123.66)
+		(width 0.8)
+		(layer "B.Cu")
+		(net 27)
+	)
+	(segment
 		(start 151.38 112.0713)
-		(end 151.38 113.5)
+		(end 163.4513 100)
+		(width 0.8)
+		(layer "B.Cu")
+		(net 27)
+	)
+	(segment
+		(start 171.7 106.3)
+		(end 171.7 112.2)
+		(width 0.8)
+		(layer "B.Cu")
+		(net 27)
+	)
+	(segment
+		(start 172.1 112.6)
+		(end 171.7 112.2)
+		(width 0.15)
+		(layer "B.Cu")
+		(net 27)
+	)
+	(segment
+		(start 171.7 112.6)
+		(end 171.7 115.1113)
+		(width 0.8)
+		(layer "B.Cu")
+		(net 27)
+	)
+	(segment
+		(start 176.83 112.6)
+		(end 171.7 112.6)
 		(width 0.8)
 		(layer "B.Cu")
@@
 		(width 0.8)
 		(layer "B.Cu")
-		(net 27)
-	)
-	(segment
-		(start 170.6387 105.2387)
-		(end 165.4 100)
-		(width 0.8)
-		(layer "B.Cu")
